Commit message: Calibrate ekf

File: example_description/robot/visual/mobile.xacro (robot description, xacro)
@@ -36,5 +36,5 @@
             <parent link="base_link"/>
             <child link="left_wheel"/>
-            <origin xyz="0 0.0845 -0.024" rpy="0 0 0"/>
+            <origin xyz="0 0.08125 -0.024" rpy="0 0 0"/>
             <axis xyz="0 1 0"/>
             <limit
@@ -47,5 +47,5 @@
             <parent link="base_link"/>
             <child link="right_wheel"/>
-            <origin xyz="0 -0.0845 -0.024" rpy="0 0 0"/>
+            <origin xyz="0 -0.08125 -0.024" rpy="0 0 0"/>
             <axis xyz="0 1 0"/>
             <limit

Commit message: .

File: example_description/robot/visual/mobile.xacro (robot description, xacro)
@@ -15,5 +15,5 @@
     <!-- Pure Visual (No dynamics) -->
     <xacro:macro name="manipulator_visual" params="">
-        <link name="base"/>
+        <link name="odom"/>
         <link name="base_link">
             <origin xyz="0 0 0" rpy="0 0 0"/>
@@ -29,5 +29,5 @@
         <!-- <link name="end_effector"/> -->
         <joint name="base_offset" type="fixed">
-            <parent link="base"/>
+            <parent link="odom"/>
             <child link="base_link"/>
             <origin xyz="0 0 0.05775" rpy="0 0 0"/>

Commit message: change URDF

File: example_description/robot/visual/mobile.xacro (robot description, xacro)
@@ -63,5 +63,5 @@
             <parent link="tilt_link"/>
             <child link="imu"/>
-            <origin xyz="0.097 0 0" rpy="0 0 0"/>
+            <origin xyz="0.0 0 0" rpy="3.14159265359 0 0"/>
         </joint>
         <!-- <joint name="end_effector_offset" type="fixed">

Commit message: chage imu frame

File: example_description/robot/visual/mobile.xacro (robot description, xacro)
@@ -63,5 +63,5 @@
             <parent link="tilt_link"/>
             <child link="imu"/>
-            <origin xyz="0.0 0 0" rpy="3.14159265359 0 0"/>
+            <origin xyz="0.0 0 0" rpy="0 0 0"/>
         </joint>
         <!-- <joint name="end_effector_offset" type="fixed">
